File: pulseFilter.kicad_pcb (KiCad board)
At the start: 2 copper layers, 72 x 47 mm, 30 parts, among them U1 TMU_3-1213, U3 NJM2903D, U4 LDK320ADU120R

Commit message: bug fix
Parts:
- removed U4: LDK320ADU120R, filter:SOT-23-3
- added U2: LDK320ADU120R, filter:SOT-23-3, F.Cu at (141.1, 93.1)
- U3: footprint Package_DIP:DIP-8_W10.16mm -> Package_DIP:DIP-8_W7.62mm
- moved U1 4.66 mm to (125.5, 90.4), turned to 90 degrees
- moved R6 2.98 mm to (170.7, 92.9)
- moved R1 2.90 mm to (166.0, 92.9)
- moved C4 2.25 mm to (146.8, 93.4)
- moved C3 1.12 mm to (137.8, 92.4)
Connections:
- U1 pad 1: GND -> 15V
- U1 pad 2: VBAT12V -> GND
- U1 pad 3: GND -> VBAT12V
- U1 pad 4: 15V -> GND
Routing:
- net VREF: track 34.1 -> 27.6 mm
- net 15V: track 10.6 -> 16.7 mm
- net VBAT12V: track 22.8 -> 27.4 mm
- net Net-(R1-Pad2): track 30.6 -> 33.8 mm
- net Net-(R4-Pad2): track 23.7 -> 26.3 mm
- net 12V: track 90.2 -> 90.8 mm
