File: pulseFilter.kicad_sch (KiCad schematic)
At the start: 21 parts, among them U1 TMU_3-1213, U3 NJM2903D, U4 LDK320ADU120R

Commit message: update
Parts:
- added C7, C8: 0, Capacitor_SMD:C_0603_1608Metric, symbol pspice:C
- added R10, R9: 0, Resistor_THT:R_Axial_DIN0204_L3.6mm_D1.6mm_P7.62mm_Horizontal, symbol Device:R_US
- C5: value 1u -> 0.1u
Connections:
- net 12V: now also RV1.3; no longer RV1.1
- net GND: now also RV1.1, C7.2, C8.2; no longer RV1.3
- net PULSE1: now also C7.1, R9.2; no longer R2.2, R5.2, U3.1 (out)
- net PULSE2: now also C8.1, R10.2; no longer R1.2, R6.2, U3.7 (out)
- new net: R2.2, R5.2, R9.1, U3.1 (out)
- new net: R1.2, R10.1, R6.2, U3.7 (out)
Other:
- moved on the sheet: C5, R1, R2, R4, R6, RV1, U3B

Commit message: to chip resistors
Parts:
- R1, R10, R2, R3, R4, R5, R6, R7, R8, R9: footprint Resistor_THT:R_Axial_DIN0204_L3.6mm_D1.6mm_P7.62mm_Horizontal -> Resistor_SMD:R_0603_1608Metric_Pad0.98x0.95mm_HandSolder
Changed lines of the file:
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@@
     (property "Reference" "R5" (id 0) (at 199.39 71.12 90))
     (property "Value" "1M" (id 1) (at 199.39 73.66 90))
-    (property "Footprint" "Resistor_THT:R_Axial_DIN0204_L3.6mm_D1.6mm_P7.62mm_Horizontal" (id 2) (at 199.644 76.454 90)
+    (property "Footprint" "Resistor_SMD:R_0603_1608Metric_Pad0.98x0.95mm_HandSolder" (id 2) (at 199.644 76.454 90)
       (effects (font (size 1.27 1.27)) hide)
     )
@@
     (property "Reference" "R6" (id 0) (at 201.93 114.3 90))
     (property "Value" "1M" (id 1) (at 201.93 116.84 90))
-    (property "Footprint" "Resistor_THT:R_Axial_DIN0204_L3.6mm_D1.6mm_P7.62mm_Horizontal" (id 2) (at 202.184 119.634 90)
+    (property "Footprint" "Resistor_SMD:R_0603_1608Metric_Pad0.98x0.95mm_HandSolder" (id 2) (at 202.184 119.634 90)
       (effects (font (size 1.27 1.27)) hide)
     )
@@
       (effects (font (size 1.27 1.27)) (justify right))
     )
-    (property "Footprint" "Resistor_THT:R_Axial_DIN0204_L3.6mm_D1.6mm_P7.62mm_Horizontal" (id 2) (at 141.224 54.356 90)
+    (property "Footprint" "Resistor_SMD:R_0603_1608Metric_Pad0.98x0.95mm_HandSolder" (id 2) (at 141.224 54.356 90)
       (effects (font (size 1.27 1.27)) hide)
     )
@@
     (property "Reference" "R10" (id 0) (at 232.41 130.81 90))
     (property "Value" "0" (id 1) (at 232.41 133.35 90))
-    (property "Footprint" "Resistor_THT:R_Axial_DIN0204_L3.6mm_D1.6mm_P7.62mm_Horizontal" (id 2) (at 232.664 136.144 90)
+    (property "Footprint" "Resistor_SMD:R_0603_1608Metric_Pad0.98x0.95mm_HandSolder" (id 2) (at 232.664 136.144 90)
       (effects (font (size 1.27 1.27)) hide)
     )
@@
     (property "Reference" "R4" (id 0) (at 190.5 128.27 90))
     (property "Value" "1k" (id 1) (at 190.5 130.81 90))
-    (property "Footprint" "Resistor_THT:R_Axial_DIN0204_L3.6mm_D1.6mm_P7.62mm_Horizontal" (id 2) (at 190.754 133.604 90)
+    (property "Footprint" "Resistor_SMD:R_0603_1608Metric_Pad0.98x0.95mm_HandSolder" (id 2) (at 190.754 133.604 90)
       (effects (font (size 1.27 1.27)) hide)
     )
@@
       (effects (font (size 1.27 1.27)) (justify left))
     )
-    (property "Footprint" "Resistor_THT:R_Axial_DIN0204_L3.6mm_D1.6mm_P7.62mm_Horizontal" (id 2) (at 218.186 129.794 90)
+    (property "Footprint" "Resistor_SMD:R_0603_1608Metric_Pad0.98x0.95mm_HandSolder" (id 2) (at 218.186 129.794 90)
       (effects (font (size 1.27 1.27)) hide)
     )
@@
       (effects (font (size 1.27 1.27)) (justify right))
     )
-    (property "Footprint" "Resistor_THT:R_Axial_DIN0204_L3.6mm_D1.6mm_P7.62mm_Horizontal" (id 2) (at 141.224 74.676 90)
+    (property "Footprint" "Resistor_SMD:R_0603_1608Metric_Pad0.98x0.95mm_HandSolder" (id 2) (at 141.224 74.676 90)
       (effects (font (size 1.27 1.27)) hide)
     )
@@
     (property "Reference" "R3" (id 0) (at 186.69 87.63 90))
     (property "Value" "1k" (id 1) (at 186.69 90.17 90))
-    (property "Footprint" "Resistor_THT:R_Axial_DIN0204_L3.6mm_D1.6mm_P7.62mm_Horizontal" (id 2) (at 186.944 92.964 90)
+    (property "Footprint" "Resistor_SMD:R_0603_1608Metric_Pad0.98x0.95mm_HandSolder" (id 2) (at 186.944 92.964 90)
       (effects (font (size 1.27 1.27)) hide)
     )
@@
       (effects (font (size 1.27 1.27)) (justify left))
     )
-    (property "Footprint" "Resistor_THT:R_Axial_DIN0204_L3.6mm_D1.6mm_P7.62mm_Horizontal" (id 2) (at 224.536 91.694 90)
+    (property "Footprint" "Resistor_SMD:R_0603_1608Metric_Pad0.98x0.95mm_HandSolder" (id 2) (at 224.536 91.694 90)
       (effects (font (size 1.27 1.27)) hide)
     )
@@
     (property "Reference" "R9" (id 0) (at 236.22 90.17 90))
     (property "Value" "0" (id 1) (at 236.22 92.71 90))
-    (property "Footprint" "Resistor_THT:R_Axial_DIN0204_L3.6mm_D1.6mm_P7.62mm_Horizontal" (id 2) (at 236.474 95.504 90)
+    (property "Footprint" "Resistor_SMD:R_0603_1608Metric_Pad0.98x0.95mm_HandSolder" (id 2) (at 236.474 95.504 90)
       (effects (font (size 1.27 1.27)) hide)
     )
@@
     )
     (path "/4dd7ea7b-9317-4033-ab6c-2f17e65acd8d"
-      (reference "R1") (unit 1) (value "1k") (footprint "Resistor_THT:R_Axial_DIN0204_L3.6mm_D1.6mm_P7.62mm_Horizontal")
+      (reference "R1") (unit 1) (value "1k") (footprint "Resistor_SMD:R_0603_1608Metric_Pad0.98x0.95mm_HandSolder")
     )
     (path "/ab5771f5-ceef-483d-8c49-faf6d9c5a400"
-      (reference "R2") (unit 1) (value "1k") (footprint "Resistor_THT:R_Axial_DIN0204_L3.6mm_D1.6mm_P7.62mm_Horizontal")
+      (reference "R2") (unit 1) (value "1k") (footprint "Resistor_SMD:R_0603_1608Metric_Pad0.98x0.95mm_HandSolder")
     )
     (path "/8adb7964-5ef8-444f-b8bc-8c1494f2f59e"
-      (reference "R3") (unit 1) (value "1k") (footprint "Resistor_THT:R_Axial_DIN0204_L3.6mm_D1.6mm_P7.62mm_Horizontal")
+      (reference "R3") (unit 1) (value "1k") (footprint "Resistor_SMD:R_0603_1608Metric_Pad0.98x0.95mm_HandSolder")
     )
     (path "/331bf168-db77-4d71-bdd6-1ce7f157e8cf"
-      (reference "R4") (unit 1) (value "1k") (footprint "Resistor_THT:R_Axial_DIN0204_L3.6mm_D1.6mm_P7.62mm_Horizontal")
+      (reference "R4") (unit 1) (value "1k") (footprint "Resistor_SMD:R_0603_1608Metric_Pad0.98x0.95mm_HandSolder")
     )
     (path "/01be7dfe-9d29-47e3-93c7-56dd9ca25c99"
-      (reference "R5") (unit 1) (value "1M") (footprint "Resistor_THT:R_Axial_DIN0204_L3.6mm_D1.6mm_P7.62mm_Horizontal")
+      (reference "R5") (unit 1) (value "1M") (footprint "Resistor_SMD:R_0603_1608Metric_Pad0.98x0.95mm_HandSolder")
     )
     (path "/0fac2c9a-167d-42f7-886d-0adf0fd0dded"
-      (reference "R6") (unit 1) (value "1M") (footprint "Resistor_THT:R_Axial_DIN0204_L3.6mm_D1.6mm_P7.62mm_Horizontal")
+      (reference "R6") (unit 1) (value "1M") (footprint "Resistor_SMD:R_0603_1608Metric_Pad0.98x0.95mm_HandSolder")
     )
     (path "/1a893a12-c79e-4641-9723-b7926fdc2423"
-      (reference "R7") (unit 1) (value "100") (footprint "Resistor_THT:R_Axial_DIN0204_L3.6mm_D1.6mm_P7.62mm_Horizontal")
+      (reference "R7") (unit 1) (value "100") (footprint "Resistor_SMD:R_0603_1608Metric_Pad0.98x0.95mm_HandSolder")
     )
     (path "/8281d564-064c-44c0-834a-3d4de1ce9e95"
-      (reference "R8") (unit 1) (value "100") (footprint "Resistor_THT:R_Axial_DIN0204_L3.6mm_D1.6mm_P7.62mm_Horizontal")
+      (reference "R8") (unit 1) (value "100") (footprint "Resistor_SMD:R_0603_1608Metric_Pad0.98x0.95mm_HandSolder")
     )
     (path "/d267101b-dd01-40aa-9afd-fee291ae65ab"
-      (reference "R9") (unit 1) (value "0") (footprint "Resistor_THT:R_Axial_DIN0204_L3.6mm_D1.6mm_P7.62mm_Horizontal")
+      (reference "R9") (unit 1) (value "0") (footprint "Resistor_SMD:R_0603_1608Metric_Pad0.98x0.95mm_HandSolder")
     )
     (path "/206d26c7-104d-4188-9c54-f475e47bc3c0"
-      (reference "R10") (unit 1) (value "0") (footprint "Resistor_THT:R_Axial_DIN0204_L3.6mm_D1.6mm_P7.62mm_Horizontal")
+      (reference "R10") (unit 1) (value "0") (footprint "Resistor_SMD:R_0603_1608Metric_Pad0.98x0.95mm_HandSolder")
     )
     (path "/97f2cf17-db9f-47bd-bc3e-82fd14c2b894"

Commit message: backup
Parts:
- added TP1: TestPoint, TestPoint:TestPoint_Loop_D1.80mm_Drill1.0mm_Beaded, symbol Connector:TestPoint
- C1, C2, C3, C4, C5, C6, C7, C8: footprint Capacitor_SMD:C_0603_1608Metric -> Capacitor_SMD:C_0603_1608Metric_Pad1.08x0.95mm_HandSolder
Connections:
- net VREF: now also TP1.1
Changed lines of the file:
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@@
       (effects (font (size 1.27 1.27)) (justify left))
     )
-    (property "Footprint" "Capacitor_SMD:C_0603_1608Metric" (id 2) (at 95.25 96.52 0)
+    (property "Footprint" "Capacitor_SMD:C_0603_1608Metric_Pad1.08x0.95mm_HandSolder" (id 2) (at 95.25 96.52 0)
       (effects (font (size 1.27 1.27)) hide)
     )
@@
       (effects (font (size 1.27 1.27)) (justify left))
     )
-    (property "Footprint" "Capacitor_SMD:C_0603_1608Metric" (id 2) (at 246.38 102.87 0)
+    (property "Footprint" "Capacitor_SMD:C_0603_1608Metric_Pad1.08x0.95mm_HandSolder" (id 2) (at 246.38 102.87 0)
       (effects (font (size 1.27 1.27)) hide)
     )
@@
       (effects (font (size 1.27 1.27)) (justify left))
     )
-    (property "Footprint" "Capacitor_SMD:C_0603_1608Metric" (id 2) (at 153.67 146.05 0)
+    (property "Footprint" "Capacitor_SMD:C_0603_1608Metric_Pad1.08x0.95mm_HandSolder" (id 2) (at 153.67 146.05 0)
       (effects (font (size 1.27 1.27)) hide)
     )
@@
       (effects (font (size 1.27 1.27)) (justify left))
     )
-    (property "Footprint" "Capacitor_SMD:C_0603_1608Metric" (id 2) (at 72.39 156.21 0)
+    (property "Footprint" "Capacitor_SMD:C_0603_1608Metric_Pad1.08x0.95mm_HandSolder" (id 2) (at 72.39 156.21 0)
       (effects (font (size 1.27 1.27)) hide)
     )
@@
     (pin "2")
   )
+  (symbol (lib_id "Connector:TestPoint") (at 153.67 139.7 0) (unit 1)
+    (in_bom yes) (on_board yes) (fields_autoplaced)
+    (property "Reference" "TP1" (id 0) (at 156.21 135.1279 0)
+      (effects (font (size 1.27 1.27)) (justify left))
+    )
+    (property "Value" "TestPoint" (id 1) (at 156.21 137.6679 0)
+      (effects (font (size 1.27 1.27)) (justify left))
+    )
+    (property "Footprint" "TestPoint:TestPoint_Loop_D1.80mm_Drill1.0mm_Beaded" (id 2) (at 158.75 139.7 0)
+      (effects (font (size 1.27 1.27)) hide)
+    )
+    (property "Datasheet" "~" (id 3) (at 158.75 139.7 0)
+      (effects (font (size 1.27 1.27)) hide)
+    )
+    (pin "1")
+  )
   (symbol (lib_name "TMU_3-1213_1") (lib_id "filter:TMU_3-1213") (at 73.66 91.44 0) (unit 1)
     (in_bom yes) (on_board yes) (fields_autoplaced)
@@
       (effects (font (size 1.27 1.27)) (justify left))
     )
-    (property "Footprint" "Capacitor_SMD:C_0603_1608Metric" (id 2) (at 213.36 59.69 0)
+    (property "Footprint" "Capacitor_SMD:C_0603_1608Metric_Pad1.08x0.95mm_HandSolder" (id 2) (at 213.36 59.69 0)
       (effects (font (size 1.27 1.27)) hide)
     )
@@
       (effects (font (size 1.27 1.27)) (justify left))
     )
-    (property "Footprint" "Capacitor_SMD:C_0603_1608Metric" (id 2) (at 243.84 143.51 0)
+    (property "Footprint" "Capacitor_SMD:C_0603_1608Metric_Pad1.08x0.95mm_HandSolder" (id 2) (at 243.84 143.51 0)
       (effects (font (size 1.27 1.27)) hide)
     )
@@
       (effects (font (size 1.27 1.27)) (justify left))
     )
-    (property "Footprint" "Capacitor_SMD:C_0603_1608Metric" (id 2) (at 124.46 96.52 0)
+    (property "Footprint" "Capacitor_SMD:C_0603_1608Metric_Pad1.08x0.95mm_HandSolder" (id 2) (at 124.46 96.52 0)
       (effects (font (size 1.27 1.27)) hide)
     )
@@
       (effects (font (size 1.27 1.27)) (justify left))
     )
-    (property "Footprint" "Capacitor_SMD:C_0603_1608Metric" (id 2) (at 57.15 156.21 0)
+    (property "Footprint" "Capacitor_SMD:C_0603_1608Metric_Pad1.08x0.95mm_HandSolder" (id 2) (at 57.15 156.21 0)
       (effects (font (size 1.27 1.27)) hide)
     )
@@
     )
     (path "/edf7992e-dc3c-4413-8610-c62be177a031"
-      (reference "C1") (unit 1) (value "1u") (footprint "Capacitor_SMD:C_0603_1608Metric")
+      (reference "C1") (unit 1) (value "1u") (footprint "Capacitor_SMD:C_0603_1608Metric_Pad1.08x0.95mm_HandSolder")
     )
     (path "/32bd7426-7861-422a-98d7-74b8498f4fbd"
-      (reference "C2") (unit 1) (value "0.1u") (footprint "Capacitor_SMD:C_0603_1608Metric")
+      (reference "C2") (unit 1) (value "0.1u") (footprint "Capacitor_SMD:C_0603_1608Metric_Pad1.08x0.95mm_HandSolder")
     )
     (path "/0231fabc-5e6e-4ec0-a2ea-67427a770bf5"
-      (reference "C3") (unit 1) (value "1u") (footprint "Capacitor_SMD:C_0603_1608Metric")
+      (reference "C3") (unit 1) (value "1u") (footprint "Capacitor_SMD:C_0603_1608Metric_Pad1.08x0.95mm_HandSolder")
     )
     (path "/d941dfff-7c2d-4ca2-8ddb-460febe38750"
-      (reference "C4") (unit 1) (value "1u") (footprint "Capacitor_SMD:C_0603_1608Metric")
+      (reference "C4") (unit 1) (value "1u") (footprint "Capacitor_SMD:C_0603_1608Metric_Pad1.08x0.95mm_HandSolder")
     )
     (path "/2586815a-f387-4297-aea5-c265c120a335"
-      (reference "C5") (unit 1) (value "0.1u") (footprint "Capacitor_SMD:C_0603_1608Metric")
+      (reference "C5") (unit 1) (value "0.1u") (footprint "Capacitor_SMD:C_0603_1608Metric_Pad1.08x0.95mm_HandSolder")
     )
     (path "/aa023a61-be9f-4a02-829c-840b474458b1"
-      (reference "C6") (unit 1) (value "0.1u") (footprint "Capacitor_SMD:C_0603_1608Metric")
+      (reference "C6") (unit 1) (value "0.1u") (footprint "Capacitor_SMD:C_0603_1608Metric_Pad1.08x0.95mm_HandSolder")
     )
     (path "/04fe31b5-d96d-403c-8706-4f01df306344"
-      (reference "C7") (unit 1) (value "0") (footprint "Capacitor_SMD:C_0603_1608Metric")
+      (reference "C7") (unit 1) (value "0") (footprint "Capacitor_SMD:C_0603_1608Metric_Pad1.08x0.95mm_HandSolder")
     )
     (path "/d158919d-829c-4fda-9973-2cb18dfb4563"
-      (reference "C8") (unit 1) (value "0") (footprint "Capacitor_SMD:C_0603_1608Metric")
+      (reference "C8") (unit 1) (value "0") (footprint "Capacitor_SMD:C_0603_1608Metric_Pad1.08x0.95mm_HandSolder")
     )
     (path "/4dd7ea7b-9317-4033-ab6c-2f17e65acd8d"
@@
       (reference "SENSOR2") (unit 1) (value "Conn_01x04_Male") (footprint "Connector_JST:JST_XA_S04B-XASK-1N-BN_1x04_P2.50mm_Horizontal")
     )
+    (path "/8bc14f00-8759-4f0c-86a5-a83fef24d964"
+      (reference "TP1") (unit 1) (value "TestPoint") (footprint "TestPoint:TestPoint_Loop_D1.80mm_Drill1.0mm_Beaded")
+    )
     (path "/92276971-2422-4512-b60c-ccaa66d0d665"

Commit message: bug fix
Parts:
- removed U4: LDK320ADU120R, filter:SOT-23-3, symbol filter:LDK320ADU120R
- added U2: LDK320ADU120R, filter:SOT-23-3, symbol filter:LDK320ADU120R
- U3: footprint Package_DIP:DIP-8_W10.16mm -> Package_DIP:DIP-8_W7.62mm
Connections:
- net 12V: now also U2.2 (OUT)
- net 15V: now also U1.1 (+Vout), U2.3 (IN); no longer U1.4 (+Vout)
- net GND: now also U1.2 (-Vout), U1.4 (Vin-), U2.1 (GND); no longer U1.1 (GND), U1.3 (-Vout)
- net VBAT12V: now also U1.3 (Vin+); no longer U1.2 (Vin)
Changed lines of the file:
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@@
     (stroke (width 0) (type default) (color 0 0 0 0))
   )
-  (wire (pts (xy 105.41 96.52) (xy 105.41 99.06))
+  (wire (pts (xy 105.41 95.25) (xy 105.41 99.06))
     (stroke (width 0) (type default) (color 0 0 0 0))
   )
@@
     (pin "2")
   )
+  (symbol (lib_name "LDK320ADU120R_2") (lib_id "filter:LDK320ADU120R") (at 113.03 88.9 0) (unit 1)
+    (in_bom yes) (on_board yes) (fields_autoplaced)
+    (property "Reference" "U2" (id 0) (at 113.03 81.28 0))
+    (property "Value" "LDK320ADU120R" (id 1) (at 113.03 83.82 0))
+    (property "Footprint" "filter:SOT-23-3" (id 2) (at 113.03 101.6 0)
+      (effects (font (size 1.27 1.27)) hide)
+    )
+    (property "Datasheet" "" (id 3) (at 113.03 88.9 0)
+      (effects (font (size 1.27 1.27)) hide)
+    )
+    (pin "1")
+    (pin "2")
+    (pin "3")
+  )
   (symbol (lib_id "Device:R_US") (at 232.41 137.16 90) (unit 1)
     (in_bom yes) (on_board yes) (fields_autoplaced)
@@
     (property "Reference" "U3" (id 0) (at 213.36 92.1893 0))
     (property "Value" "NJM2903D" (id 1) (at 213.36 94.7293 0))
-    (property "Footprint" "Package_DIP:DIP-8_W10.16mm" (id 2) (at 193.04 90.17 0)
+    (property "Footprint" "Package_DIP:DIP-8_W7.62mm" (id 2) (at 193.04 90.17 0)
       (effects (font (size 1.27 1.27)) hide)
     )
@@
     (property "Reference" "U3" (id 0) (at 206.375 125.73 0))
     (property "Value" "NJM2903D" (id 1) (at 206.375 128.27 0))
-    (property "Footprint" "Package_DIP:DIP-8_W10.16mm" (id 2) (at 196.85 130.81 0)
+    (property "Footprint" "Package_DIP:DIP-8_W7.62mm" (id 2) (at 196.85 130.81 0)
       (effects (font (size 1.27 1.27)) hide)
     )
@@
     (pin "1")
   )
-  (symbol (lib_name "TMU_3-1213_1") (lib_id "filter:TMU_3-1213") (at 73.66 91.44 0) (unit 1)
+  (symbol (lib_id "filter:TMU_3-1213") (at 73.66 91.44 0) (unit 1)
     (in_bom yes) (on_board yes) (fields_autoplaced)
     (property "Reference" "U1" (id 0) (at 74.295 82.55 0))
     (property "Value" "TMU_3-1213" (id 1) (at 74.295 85.09 0))
-    (property "Footprint" "filter:TRACO POWER DCDC" (id 2) (at 73.66 91.44 0)
+    (property "Footprint" "filter:TRACO POWER DCDC" (id 2) (at 74.93 99.06 0)
       (effects (font (size 1.27 1.27)) hide)
     )
@@
     (pin "2")
   )
-  (symbol (lib_id "filter:LDK320ADU120R") (at 113.03 90.17 0) (unit 1)
-    (in_bom yes) (on_board yes) (fields_autoplaced)
-    (property "Reference" "U4" (id 0) (at 113.03 80.01 0))
-    (property "Value" "LDK320ADU120R" (id 1) (at 113.03 82.55 0))
-    (property "Footprint" "filter:SOT-23-3" (id 2) (at 113.03 85.09 0))
-    (property "Datasheet" "" (id 3) (at 113.03 90.17 0)
-      (effects (font (size 1.27 1.27)) hide)
-    )
-    (pin "1")
-    (pin "2")
-    (pin "3")
-  )
   (symbol (lib_id "Device:R_US") (at 236.22 96.52 90) (unit 1)
     (in_bom yes) (on_board yes) (fields_autoplaced)
@@
       (reference "TP1") (unit 1) (value "TestPoint") (footprint "TestPoint:TestPoint_Loop_D1.80mm_Drill1.0mm_Beaded")
     )
-    (path "/92276971-2422-4512-b60c-ccaa66d0d665"
+    (path "/8c0f0bf9-ddba-4307-87e9-3dcf1a39b5eb"
       (reference "U1") (unit 1) (value "TMU_3-1213") (footprint "filter:TRACO POWER DCDC")
     )
+    (path "/1c7ce082-fab4-4e06-863e-946528af2cf7"
+      (reference "U2") (unit 1) (value "LDK320ADU120R") (footprint "filter:SOT-23-3")
+    )
     (path "/262fbede-08f0-4dfb-ac0e-d93901f45227"
-      (reference "U3") (unit 1) (value "NJM2903D") (footprint "Package_DIP:DIP-8_W10.16mm")
+      (reference "U3") (unit 1) (value "NJM2903D") (footprint "Package_DIP:DIP-8_W7.62mm")
     )
     (path "/3432dd11-6b9f-4f85-ba9d-b1fcdcd8e354"
-      (reference "U3") (unit 2) (value "NJM2903D") (footprint "Package_DIP:DIP-8_W10.16mm")
-    )
-    (path "/d19c47c4-c88a-4187-84a8-2abc0d294422"
-      (reference "U4") (unit 1) (value "LDK320ADU120R") (footprint "filter:SOT-23-3")
+      (reference "U3") (unit 2) (value "NJM2903D") (footprint "Package_DIP:DIP-8_W7.62mm")
     )
     (path "/538f08f4-c749-456f-918e-e183a59dd238"
